Commit message: Custom Parameters Added

File: config/robot.urdf.xacro (robot description, xacro)
@@ -30,5 +30,5 @@
   <joint name="navsat_joint" type="fixed">
     <parent link="chassis_link" />
-    <child link="navsat_link" />
+    <child link="gps" />
     <origin xyz="0 0 0" rpy="0 0 0" />
   </joint>
